Commit message: Add imu to sim

File: diffbot_description/urdf/diffbot.urdf.xacro (robot description, xacro)
@@ -50,4 +50,7 @@
                    enable_gpu="${sensor_prop['laser']['enable_gpu']}">
   </xacro:laser>
+  <xacro:imu_sensor parent_link="base_link" sensor_prop="${sensor_prop}">
+    <joint_origin xyz="0 0 0" rpy="0 0 0"/>
+  </xacro:imu_sensor>
   <!-- Gazebo -->
   <xacro:gazebo_ros_control robotNamespace="/diffbot">

File: diffbot_description/urdf/include/common_sensors.xacro (robot description, xacro)
@@ -14,21 +14,21 @@
   <link name="${prefix}_laser_link">
     <xacro:if value="${mesh != '' }" >
-    <visual>
-      <origin xyz="0 0 0" rpy="0 0 ${pi}"/>
-      <geometry>
-        <mesh filename="package://${package_name}/meshes/sensors/${mesh}" />
-      </geometry>
-      <material name="dark_grey"/>
-    </visual>
-  </xacro:if>
-  <xacro:if value="${mesh == '' }" >
-    <visual>
-      <origin xyz="0 0 0" rpy="0 0 0"/>
-        <geometry>
-        <cylinder radius="${sensor_prop['laser']['radius']}" length="${sensor_prop['laser']['length']}"/>
-      </geometry>
-      <material name="red"/>
-    </visual>
-  </xacro:if>
+      <visual>
+        <origin xyz="0 0 0" rpy="0 0 ${pi}"/>
+        <geometry>
+          <mesh filename="package://${package_name}/meshes/sensors/${mesh}" />
+        </geometry>
+        <material name="dark_grey"/>
+      </visual>
+    </xacro:if>
+    <xacro:if value="${mesh == '' }" >
+      <visual>
+        <origin xyz="0 0 0" rpy="0 0 0"/>
+          <geometry>
+          <cylinder radius="${sensor_prop['laser']['radius']}" length="${sensor_prop['laser']['length']}"/>
+        </geometry>
+        <material name="red"/>
+      </visual>
+    </xacro:if>
     <collision>
       <origin xyz="0 0 0" rpy="0 0 0"/>
@@ -190,7 +190,8 @@
     <xacro:if value="${mesh == '' }" >
       <visual>
-        <origin xyz="0 0 0" rpy="0 0 0"/>
-        <geometry>
-          <cylinder radius="${sensor_prop['imu']['radius']}" length="${sensor_prop['imu']['length']}"/>
+        <origin xyz="-0.07 0 0.01" rpy="0 0 0"/>
+        <geometry>
+          <!-- <cylinder radius="${sensor_prop['imu']['radius']}" length="${sensor_prop['imu']['length']}"/> -->
+          <box size="${sensor_prop['imu']['size']['x']} ${sensor_prop['imu']['size']['y']} ${sensor_prop['imu']['size']['z']}"/>
         </geometry>
         <material name="red"/>
@@ -206,5 +207,5 @@
                        x="${sensor_prop['imu']['size']['x']}"
                        y="${sensor_prop['imu']['size']['y']}"
-                       z="${sensor_prop['imu']['size']['y']}" />
+                       z="${sensor_prop['imu']['size']['z']}" />
     <!-- Todo delete visual>
       <origin xyz="0 0 0" rpy="0 0 0"/>
@@ -228,17 +229,34 @@
     <child link="imu_link"/>
   </joint>
-  <gazebo reference="imu_link">
+  <!-- <gazebo reference="imu_link">
     <sensor type="imu" name="my_imu">
     <always_on>true</always_on>
-    <!-- Publish at 30 hz -->
     <update_rate>30</update_rate>
     <plugin name="my_imu_plugin" filename="libgazebo_ros_imu_sensor.so">
       <ros>
-        <!-- Will publish to /imu/data -->
         <namespace>/imu</namespace>
         <argument>~/out:=data</argument>
       </ros>
-      <!-- frame_name ommited, will be "my_link" -->
     </plugin>
+    </sensor>
+  </gazebo> -->
+  <gazebo reference="imu_link">
+    <gravity>true</gravity>
+    <sensor name="my_imu" type="imu">
+      <always_on>true</always_on>
+      <update_rate>100</update_rate>
+      <visualize>true</visualize>
+      <topic>__default_topic__</topic>
+      <plugin filename="libgazebo_ros_imu_sensor.so" name="imu_plugin">
+        <topicName>imu</topicName>
+        <bodyName>imu_link</bodyName>
+        <updateRateHZ>100.0</updateRateHZ>
+        <gaussianNoise>0.05</gaussianNoise>
+        <xyzOffset>0 0 0</xyzOffset>
+        <rpyOffset>0 0 0</rpyOffset>
+        <frameName>imu_link</frameName>
+        <initialOrientationAsReference>false</initialOrientationAsReference>
+      </plugin>
+      <pose>0 0 0 0 0 0</pose>
     </sensor>
   </gazebo>
